File: Lab1.sch (KiCad schematic (older format))
At the start: 38 parts, among them J1 USB_OTG, J2 SWD, SW1 Reset, SW2 Reset, U1 PMW3389, U2 AP2125N-3.3TRG, U3 MIC5235YM5-TR, U4 STM32F411RETx, Y1 16Mhz

Commit message: Add files via upload
Parts:
- removed SW1: Reset, Button_Switch_SMD:SW_SPST_B3U-1000P, symbol Switch:SW_Push
- removed TP5: TestPoint, TestPoint:TestPoint_Pad_1.5x1.5mm, symbol Connector:TestPoint
- added C16, C19: 10u, Capacitor_SMD:C_0805_2012Metric_Pad1.18x1.45mm_HandSolder, symbol Device:C_Small
- added C17, C18, C20: 100n, Capacitor_SMD:C_0805_2012Metric_Pad1.18x1.45mm_HandSolder, symbol Device:C_Small
- added C21: 4u7, Capacitor_SMD:C_0805_2012Metric_Pad1.18x1.45mm_HandSolder, symbol Device:C_Small
- added D2, D3: Indicator LED, LED_SMD:LED_1206_3216Metric, symbol LED:IR26-21C_L110_TR8
- added U5: USBLC6-2SC6, Package_TO_SOT_SMD:SOT-23-6, symbol Power_Protection:USBLC6-2SC6
- C3: value 4u7 -> 1u
- C4: value 4u7 -> 2.2u
- C8: value 0.1uF -> 100n
- R2: value 10k -> 5.6k
- R3: value 18k -> 10k
- U1: footprint (none) -> Battery:PMW3389
Connections:
- net +3V3: now also U1.5 (VDDIO), C19.2, C20.2, D2.2 (A)
- net +5V: now also C8.2
- net BOOT0: now also JP1.1 (A), R4.1
- net GND: now also C16.2, C17.2, C18.2, C19.1, C20.1, C21.2, D2.1 (K), D3.1 (K), U5.2 (GND); no longer C8.2
- net NRST: no longer C8.1
- net VDD: now also U1.4 (VDD), C16.1, C17.1, D3.2 (A)
- net Motion: now reaches U4.24 (PC4)
- net Motion: now also U1.9 (MOTION)
- net at U1.3 (VDCPIX): now also C18.1, C21.1
- net 5V_LED: now reaches D1.2 (A), R1.1
- net D+ renamed IN_D+
- net IN_D+: now also U5.1 (I/O1); no longer U4.45 (PA12)
- net D- renamed IN_D-
- net IN_D-: now also U5.3 (I/O2); no longer U4.44 (PA11)
- new net: C8.1, U5.5 (VBUS)
- new net OUT_D+: U4.45 (PA12), U5.6 (I/O1)
- new net OUT_D-: U4.44 (PA11), U5.4 (I/O2)
- no-connect marks 51 -> 47
Other:
- note added: "IR_SENSOR"
- note added: "LEDS"
- note added: "MICRO CONTROLLER"
- note added: "Micro Control Buttons"
- note added: "POWER MANAGEMENT"
- note added: "SWD"
- note removed: "MCU"
- moved on the sheet: C1, C15, C2, C3, C4, D1, J1, J2, JP1, R1, R2, R3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
